Commit message: Migration Gazebo Classic to Gazebo Sim Harmonic, Package Axioma Teleop GUI, Rewrite documentation from Spanish to English

File: src/axioma_description/urdf/axioma.urdf (robot description, URDF)
Before this commit: robot axioma_v2, 7 links, 6 joints
Links:
- link base_link: geometry collision mesh filename=package://axioma_description/meshes/collision/chasis.dae scale=1 1 1; visual mesh filename=package://axioma_description/meshes/visual/chasis.stl scale=1 1 1
- link wheel_1: geometry collision cylinder length=0.03 radius=0.0381; visual mesh filename=package://axioma_description/meshes/visual/llanta.stl scale=1 1 1
- link wheel_2: geometry collision cylinder length=0.03 radius=0.0381; visual mesh filename=package://axioma_description/meshes/visual/llanta.stl scale=1 1 1
- link wheel_3: geometry collision cylinder length=0.03 radius=0.0381; visual mesh filename=package://axioma_description/meshes/visual/llanta.stl scale=1 1 1
- link wheel_4: geometry collision cylinder length=0.03 radius=0.0381; visual mesh filename=package://axioma_description/meshes/visual/llanta.stl scale=1 1 1

Commit message: fix:完善基础配置使得各项功能正常运行

File: src/axioma_description/urdf/axioma.urdf (robot description, URDF)
Before this commit: robot axioma_v2, 7 links, 6 joints
Links:
- link imu_link: geometry collision box size=0.02 0.02 0.01; visual box size=0.02 0.02 0.01
